File: examples/Many-Vias/Many-Vias.kicad_pcb (KiCad board)
At the start: 4 copper layers, 17 x 40 mm, 2 parts, among them J1 IN, J2 OUT

Commit message: Update demo project
Parts:
- added R1: 10, Resistor_SMD:R_4020_10251Metric, B.Cu at (101.0, 86.2)
Connections:
- J1 pad 1: /NET -> /IN
- J2 pad 1: /NET -> /OUT
Routing:
- net /OUT: vias 0 -> 21
- net /NET: vias 42 -> 0
- net /IN: vias 0 -> 21
- added copper zone on B.Cu, net /IN
- added copper zone on F.Cu, net /IN
- added copper zone on In1.Cu, net /IN
- added copper zone on In2.Cu, net /IN
- added copper zone on B.Cu, net /OUT
- added copper zone on F.Cu, net /OUT
- added copper zone on In1.Cu, net /OUT
- added copper zone on In2.Cu, net /OUT
- removed copper zone on B.Cu, net /NET
- removed copper zone on F.Cu, net /NET
- removed copper zone on In1.Cu, net /NET
- removed copper zone on In2.Cu, net /NET
