File: examples/Many-Vias/Many-Vias.kicad_sch (KiCad schematic)
At the start: 2 parts, among them J1 IN, J2 OUT

Commit message: Update demo project
Parts:
- added R1: 10, Resistor_SMD:R_4020_10251Metric, symbol Device:R
Connections:
- net NET renamed IN
- net IN: now also R1.1; no longer J2.1 (Pin_1)
- new net OUT: J2.1 (Pin_1), R1.2
Changed lines of the file:
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@@
 	(wire
 		(pts
-			(xy 104.14 85.09) (xy 127 85.09)
+			(xy 104.14 85.09) (xy 111.76 85.09)
 		)
 		(stroke
@@
 		)
 	)
-	(label "NET"
-		(at 114.3 85.09 0)
+	(wire
+		(pts
+			(xy 119.38 85.09) (xy 127 85.09)
+		)
+		(stroke
+			(width 0)
+			(type default)
+		)
+	)
+	(label "OUT"
+		(at 121.92 85.09 0)
+		(effects
+			(font
+				(size 1.27 1.27)
+			)
+			(justify left bottom)
+		)
+	)
+	(label "IN"
+		(at 106.68 85.09 0)
 		(effects
 			(font
@@
 					(unit 1)
 				)
+			)
+		)
+	)
+	(symbol
+		(lib_id "Device:R")
+		(at 115.57 85.09 90)
+		(unit 1)
+		(body_style 1)
+		(exclude_from_sim no)
+		(in_bom yes)
+		(on_board yes)
+		(in_pos_files yes)
+		(dnp no)
+		(fields_autoplaced yes)
+		(property "Reference" "R1"
+			(at 115.57 78.74 90)
+			(show_name no)
+			(do_not_autoplace no)
+			(effects
+				(font
+					(size 1.27 1.27)
+				)
+			)
+		)
+		(property "Value" "10"
+			(at 115.57 81.28 90)
+			(show_name no)
+			(do_not_autoplace no)
+			(effects
+				(font
+					(size 1.27 1.27)
+				)
+			)
+		)
+		(property "Footprint" "Resistor_SMD:R_4020_10251Metric"
+			(at 115.57 86.868 90)
+			(hide yes)
+			(show_name no)
+			(do_not_autoplace no)
+			(effects
+				(font
+					(size 1.27 1.27)
+				)
+			)
+		)
+		(property "Datasheet" ""
+			(at 115.57 85.09 0)
+			(hide yes)
+			(show_name no)
+			(do_not_autoplace no)
+			(effects
+				(font
+					(size 1.27 1.27)
+				)
+			)
+		)
+		(property "Description" "Resistor"
+			(at 115.57 85.09 0)
+			(hide yes)
+			(show_name no)
+			(do_not_autoplace no)
+			(effects
+				(font
+					(size 1.27 1.27)
+				)
+			)
+		)
+		(pin "2"
+		)
+		(pin "1"
+		)
+		(instances
+			(project "Many-Vias"
+				(path "/6592b525-9462-4d1e-999d-0403060b3547"
+					(reference "R1")
+					(unit 1)
+				)
